File: HM_MAIN_ESP32-01/HM_MAIN_ESP32-01.kicad_pcb (KiCad board)
At the start: 2 copper layers, 59.1 x 46.7 mm, 3 parts, among them J2 Conn_02x19_Odd_Even, M1 ESP32-DEVKITV1

Commit message: adicionado painel
Connections:
- M1 pad GND@2: GND -> unconnected-(M1-GND-PadGND@2)
Changed lines of the file:
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@@
   (net 37 "unconnected-(J2-Pin_30-Pad30)")
   (net 38 "unconnected-(M1-Pad3V3)")
+  (net 39 "unconnected-(M1-GND-PadGND@2)")
   (footprint "Ben_modules:ESP32-DEVKITV1" (layer "F.Cu")
     (at 99.15 72.85)
-    (property "Sheetfile" "HM_ESP32-01.kicad_sch")
+    (property "Sheetfile" "HM_MAIN_ESP32-01.kicad_sch")
     (property "Sheetname" "")
     (attr exclude_from_pos_files)
@@
       (net 21 "GND") (pinfunction "GND") (pintype "bidirectional"))
     (pad "GND@2" thru_hole oval (at -13.97762 12.2682) (size 1.5 3) (drill 1) (layers "*.Cu" "*.Mask")
-      (net 21 "GND") (pinfunction "GND") (pintype "bidirectional"))
+      (net 39 "unconnected-(M1-GND-PadGND@2)") (pinfunction "GND") (pintype "bidirectional"))
     (pad "VIN" thru_hole oval (at -16.51762 -13.13434) (size 1.5 3) (drill 1) (layers "*.Cu" "*.Mask")
       (net 2 "Net-(D1-K)") (pinfunction "VIN") (pintype "bidirectional"))
@@
     (descr "Diode, DO-41_SOD81 series, Axial, Horizontal, pin pitch=10.16mm, , length*diameter=5.2*2.7mm^2, , http://www.diodes.com/_files/packages/DO-41%20(Plastic).pdf")
     (tags "Diode DO-41_SOD81 series Axial Horizontal pin pitch 10.16mm  length 5.2mm diameter 2.7mm")
-    (property "Sheetfile" "HM_ESP32-01.kicad_sch")
+    (property "Sheetfile" "HM_MAIN_ESP32-01.kicad_sch")
     (property "Sheetname" "")
     (property "Sim.Device" "D")
@@
     (tags "Through hole angled pin header THT 2x19 2.54mm double row")
     (property "Alias" "MAIN")
-    (property "Sheetfile" "HM_ESP32-01.kicad_sch")
+    (property "Sheetfile" "HM_MAIN_ESP32-01.kicad_sch")
     (property "Sheetname" "")
     (property "ki_description" "Generic connector, double row, 02x19, odd/even pin numbering scheme (row 1 odd numbers, row 2 even numbers), script generated (kicad-library-utils/schlib/autogen/connector/)")
